File: PCB/stage-controller/enc_axis.kicad_sch (KiCad schematic)
At the start: 18 parts, among them U16 TMC4361A-LA

Commit message: Finalise part numbers and I2C pullup
Complete mouser part numbers. Added pullup for I2C connector.
Parts:
- C34, C35, C36, C37, C38: Mouser 80-C603C104K5RAC3121 -> 810-C1608X7R1H104KEP
- C9: Mouser (none) -> 810-C1608X7R1H104KEP
- U10: Mouser (none) -> 595-AM26LS32ACPWR
- U7: Mouser (none) -> 538-52745-1197
Connections:
- net SAFETY renamed ESTOP
Other:
- note added: "Encoder & Tape link"
Changed lines of the file:
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@@
     (effects (font (size 1.27 1.27)) (justify left top))
+  )
+  (text "Encoder & Tape link" (at 31.242 69.85 0)
+    (effects (font (size 1.27 1.27)) (justify left bottom) (href "https://www.rls.si/eng/rlc2ic-miniature-linear-and-rotary-pcb-level-incremental-magnetic-encoder?partNumbers=RLC2ICA13BB13A00%2CMS05DM210CM027"))
   )
   (text "to linear axis\n" (at 243.6876 109.1438 90)
@@
     (effects (font (size 1.27 1.27)) (justify left bottom))
   )
-  (global_label "SAFETY" (shape input) (at 178.4096 115.062 0) (fields_autoplaced)
+  (global_label "ESTOP" (shape input) (at 178.4096 115.062 0) (fields_autoplaced)
     (effects (font (size 1.27 1.27)) (justify left))
-    (property "Intersheetrefs" "${INTERSHEET_REFS}" (at 187.9073 115.062 0)
+    (property "Intersheetrefs" "${INTERSHEET_REFS}" (at 187.242 115.062 0)
       (effects (font (size 1.27 1.27)) (justify left) hide)
     )
@@
     )
     (property "Datasheet" "https://www.molex.com/webdocs/datasheets/pdf/en-us/0527451197_FFC_FPC_CONNECTORS.pdf" (at 50.2412 110.6678 0)
+      (effects (font (size 1.27 1.27)) hide)
+    )
+    (property "Mouser" "538-52745-1197" (at 50.2412 110.6678 0)
       (effects (font (size 1.27 1.27)) hide)
     )
@@
       (effects (font (size 1.27 1.27)) hide)
     )
-    (property "Mouser" "80-C603C104K5RAC3121" (at 116.7892 79.8322 0)
+    (property "Mouser" "810-C1608X7R1H104KEP" (at 116.7892 79.8322 0)
       (effects (font (size 1.27 1.27)) hide)
     )
@@
       (effects (font (size 1.27 1.27)) hide)
     )
-    (property "Datasheet" "~" (at 186.5376 105.9688 0)
+    (property "Datasheet" "https://nl.mouser.com/datasheet/2/445/150080RS75000-3084988.pdf" (at 186.5376 105.9688 0)
       (effects (font (size 1.27 1.27)) hide)
     )
@@
     )
     (property "Datasheet" "https://www.ti.com/lit/ds/symlink/am26ls32ac.pdf?ts=1680896189222&ref_url=https%253A%252F%252Fwww.ti.com%252Finterface%252Frs-485-rs-422%252Fproducts.html" (at 87.5792 113.0046 0)
+      (effects (font (size 1.27 1.27)) hide)
+    )
+    (property "Mouser" "595-AM26LS32ACPWR" (at 87.5792 113.0046 0)
       (effects (font (size 1.27 1.27)) hide)
     )
@@
       (effects (font (size 1.27 1.27)) hide)
     )
-    (property "Mouser" "80-C603C104K5RAC3121" (at 139.2267 79.8322 0)
+    (property "Mouser" "810-C1608X7R1H104KEP" (at 139.2267 79.8322 0)
       (effects (font (size 1.27 1.27)) hide)
     )
@@
       (effects (font (size 1.27 1.27)) hide)
     )
-    (property "Mouser" "80-C603C104K5RAC3121" (at 132.1308 79.8322 0)
+    (property "Mouser" "810-C1608X7R1H104KEP" (at 132.1308 79.8322 0)
       (effects (font (size 1.27 1.27)) hide)
     )
@@
       (effects (font (size 1.27 1.27)) hide)
     )
-    (property "Mouser" "80-C603C104K5RAC3121" (at 113.0808 79.8322 0)
+    (property "Mouser" "810-C1608X7R1H104KEP" (at 113.0808 79.8322 0)
       (effects (font (size 1.27 1.27)) hide)
     )
@@
       (effects (font (size 1.27 1.27)) hide)
     )
-    (property "Mouser" "80-C603C104K5RAC3121" (at 135.699 79.8322 0)
+    (property "Mouser" "810-C1608X7R1H104KEP" (at 135.699 79.8322 0)
       (effects (font (size 1.27 1.27)) hide)
     )
@@
       (effects (font (size 1.27 1.27)) hide)
     )
+    (property "Mouser" "810-C1608X7R1H104KEP" (at 101.2444 93.8022 0)
+      (effects (font (size 1.27 1.27)) hide)
+    )

Commit message: Update PCB files
Pre-removal and submodule reorganisation
Parts:
- C17, C5: Mouser 810-C2012X7S1E106125 -> 810-C2012X5R1H106K12
Changed lines of the file:
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@@
       (effects (font (size 1.27 1.27)) hide)
     )
-    (property "Datasheet" "~" (at 116.7892 79.8322 0)
+    (property "Datasheet" "https://product.tdk.com/system/files/dam/doc/product/capacitor/ceramic/mlcc/catalog/mlcc_automotive_epoxy_en.pdf" (at 116.7892 79.8322 0)
       (effects (font (size 1.27 1.27)) hide)
     )
@@
       (effects (font (size 1.27 1.27)) hide)
     )
-    (property "Datasheet" "~" (at 139.2267 79.8322 0)
+    (property "Datasheet" "https://product.tdk.com/system/files/dam/doc/product/capacitor/ceramic/mlcc/catalog/mlcc_automotive_epoxy_en.pdf" (at 139.2267 79.8322 0)
       (effects (font (size 1.27 1.27)) hide)
     )
@@
       (effects (font (size 1.27 1.27)) hide)
     )
-    (property "Datasheet" "~" (at 132.1308 79.8322 0)
+    (property "Datasheet" "https://product.tdk.com/system/files/dam/doc/product/capacitor/ceramic/mlcc/catalog/mlcc_automotive_epoxy_en.pdf" (at 132.1308 79.8322 0)
       (effects (font (size 1.27 1.27)) hide)
     )
@@
       (effects (font (size 1.27 1.27)) hide)
     )
-    (property "Mouser" "810-C2012X7S1E106125" (at 70.104 127.1778 0)
+    (property "Mouser" "810-C2012X5R1H106K12" (at 70.104 127.1778 0)
       (effects (font (size 1.27 1.27)) hide)
     )
@@
       (effects (font (size 1.27 1.27)) hide)
     )
-    (property "Datasheet" "~" (at 113.0808 79.8322 0)
+    (property "Datasheet" "https://product.tdk.com/system/files/dam/doc/product/capacitor/ceramic/mlcc/catalog/mlcc_automotive_epoxy_en.pdf" (at 113.0808 79.8322 0)
       (effects (font (size 1.27 1.27)) hide)
     )
@@
       (effects (font (size 1.27 1.27)) hide)
     )
-    (property "Mouser" "810-C2012X7S1E106125" (at 212.1408 81.5594 0)
+    (property "Mouser" "810-C2012X5R1H106K12" (at 212.1408 81.5594 0)
       (effects (font (size 1.27 1.27)) hide)
     )
@@
       (effects (font (size 1.27 1.27)) hide)
     )
-    (property "Datasheet" "~" (at 135.699 79.8322 0)
+    (property "Datasheet" "https://product.tdk.com/system/files/dam/doc/product/capacitor/ceramic/mlcc/catalog/mlcc_automotive_epoxy_en.pdf" (at 135.699 79.8322 0)
       (effects (font (size 1.27 1.27)) hide)
     )
@@
       (effects (font (size 1.27 1.27)) hide)
     )
-    (property "Datasheet" "~" (at 101.2444 93.8022 0)
-      (effects (font (size 1.27 1.27)) hide)
-    )
+    (property "Datasheet" "https://product.tdk.com/system/files/dam/doc/product/capacitor/ceramic/mlcc/catalog/mlcc_automotive_epoxy_en.pdf" (at 101.2444 93.8022 0)
+      (effects (font (size 1.27 1.27)) hide)
+    )
